File: main_board.brd (EAGLE design)
At the start: 44.4 x 36.5 mm, 25 parts, among them IC1 MC34063AD, IC2 LM358N

Commit message: routed pcb
Parts:
- moved C1 0.65 mm to (37.5, 21.5)
Routing:
- net N$4: track 0.00 -> 79.0 mm
- net GND: track 0.00 -> 67.8 mm, vias 0 -> 2
- net VCC: track 0.00 -> 56.6 mm
- net N$10: track 0.00 -> 29.6 mm
- net N$5: track 0.00 -> 26.2 mm
- net N$1: track 0.00 -> 22.3 mm
- net N$3: track 0.00 -> 20.2 mm
- net N$6: track 0.00 -> 20.0 mm
- net N$8: track 0.00 -> 15.6 mm
- net N$7: track 0.00 -> 14.2 mm
- net N$9: track 0.00 -> 8.87 mm
- net N$2: track 0.00 -> 2.72 mm
- net N$12: track 0.00 -> 2.65 mm
Other:
- board size 44.4 x 36.5 mm -> 44.4 x 36.9 mm

Commit message: pcb completed
Parts:
- turned JP2 to 270 degrees
Routing:
- net GND: track 67.8 -> 66.7 mm
- net VCC: track 56.6 -> 55.7 mm
Changed lines of the file:
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@@
 <element name="IC2" library="linear" package="DIL08" value="LM358N" x="24.13" y="16.51" rot="R180"/>
 <element name="JP1" library="pinhead" package="1X02" value="MOTOR" x="26.67" y="33.02" rot="R180"/>
-<element name="JP2" library="pinhead" package="1X02" value="POWER" x="2.54" y="11.43" rot="R90"/>
+<element name="JP2" library="pinhead" package="1X02" value="POWER" x="2.54" y="11.43" rot="R270"/>
 <element name="R1" library="resistor" package="R0805" value="1" x="33.02" y="6.35" rot="R90"/>
 <element name="R10" library="pot" package="CA6V" value="15k" x="8.89" y="5.08" rot="R90"/>
@@
 <wire x1="15.06" y1="14.056" x2="15.24" y2="14.01" width="0.8" layer="1"/>
 <wire x1="11.4456" y1="14.056" x2="11.43" y2="13.97" width="0.8" layer="1"/>
-<wire x1="7.6304" y1="10.2408" x2="2.6104" y2="10.2408" width="0.8" layer="16"/>
-<wire x1="11.2448" y1="13.8552" x2="7.6304" y2="10.2408" width="0.8" layer="16"/>
-<wire x1="2.6104" y1="10.2408" x2="2.54" y2="10.16" width="0.8" layer="16"/>
 <wire x1="11.2448" y1="13.8552" x2="11.43" y2="13.97" width="0.8" layer="16"/>
 <wire x1="27.9112" y1="10.04" x2="27.9112" y2="12.6504" width="0.8" layer="16"/>
@@
 <wire x1="27.9112" y1="12.6504" x2="27.94" y2="12.7" width="0.8" layer="16"/>
 <wire x1="11.6464" y1="13.6544" x2="11.43" y2="13.97" width="0.8" layer="16"/>
+<wire x1="11.43" y1="13.97" x2="3.81" y2="13.97" width="0.8" layer="16"/>
+<wire x1="3.81" y1="13.97" x2="2.54" y2="12.7" width="0.8" layer="16"/>
 </signal>
 <signal name="N$1">
@@
 <wire x1="36.7464" y1="19.8792" x2="34.5376" y2="17.6704" width="0.8" layer="1"/>
 <wire x1="34.5376" y1="17.6704" x2="34.29" y2="17.46" width="0.8" layer="1"/>
-<wire x1="5.2208" y1="10.2408" x2="7.8312" y2="10.2408" width="0.8" layer="1"/>
-<wire x1="2.6104" y1="12.8512" x2="5.2208" y2="10.2408" width="0.8" layer="1"/>
-<wire x1="7.8312" y1="10.2408" x2="7.94" y2="10.16" width="0.8" layer="1"/>
-<wire x1="2.6104" y1="12.8512" x2="2.54" y2="12.7" width="0.8" layer="1"/>
+<wire x1="7.94" y1="10.16" x2="7.8312" y2="10.2408" width="0.8" layer="1"/>
 <wire x1="11.4456" y1="19.076" x2="15.06" y2="19.076" width="0.8" layer="1"/>
 <wire x1="15.06" y1="19.076" x2="15.24" y2="19.01" width="0.8" layer="1"/>
@@
 <via x="25.7024" y="25.7024" extent="1-16" drill="0.6096"/>
 <via x="31.5256" y="19.076" extent="1-16" drill="0.6096"/>
+<wire x1="2.54" y1="10.2408" x2="2.54" y2="10.16" width="0.8" layer="1"/>
+<wire x1="7.8312" y1="10.2408" x2="2.54" y2="10.2408" width="0.8" layer="1"/>
 </signal>
 <signal name="N$2">
